Commit message: add inertia macros and inertial tags to links

File: my_robot_description/urdf/common_properties.xacro (robot description, xacro)
@@ -12,3 +12,26 @@
     <color rgba="0 0 0.5 1" />
   </material>
+  <!-- Inertia macro -->
+  <xacro:macro name="box_inertia" params="m l w h xyz rpy">
+    <inertial>
+      <origin xyz="${xyz}" rpy="${rpy}"/>
+      <mass value="${m}"/>
+      <!-- <inertia ixx="${(m/12.0) * (h*h + l*l)}" ixy="0.0" ixz="0.0" iyy="${(m/12.0) * (w*w + h*h)}" iyz="0.0" izz="${(m/12.0) * (w*w + l*l)}" /> -->
+      <inertia ixx="${(m/12.0) * (w*w + h*h)}" ixy="0.0" ixz="0.0" iyy="${(m/12.0) * (h*h + l*l)}" iyz="0.0" izz="${(m/12.0) * (w*w + l*l)}" />
+    </inertial>
+  </xacro:macro>
+  <xacro:macro name="cylinder_inertia" params="m radius length xyz rpy">
+    <inertial>
+      <origin xyz="${xyz}" rpy="${rpy}"/>
+      <mass value="${m}"/>
+      <inertia ixx="${(m/12.0) * (3 * radius * radius + length * length) }" ixy="0.0" ixz="0.0" iyy="${(m/12.0) * (3 * radius * radius + length * length) }" iyz="0.0" izz="${m/2.0 * (radius * radius) }" />
+    </inertial>
+  </xacro:macro>
+  <xacro:macro name="sphere_inertia" params="m radius xyz rpy">
+    <inertial>
+      <origin xyz="${xyz}" rpy="${rpy}"/>
+      <mass value="${m}"/>
+      <inertia ixx="${(2 * m)/5.0 * (radius * radius)}" ixy="0.0" ixz="0.0" iyy="${(2 * m)/5.0 * (radius * radius)}" iyz="0.0" izz="${(2 * m)/5.0 * (radius * radius)}" />
+    </inertial>
+  </xacro:macro>
 </robot>

File: my_robot_description/urdf/mobile_base.xacro (robot description, xacro)
@@ -22,4 +22,6 @@
       <material name="blue" />
     </visual>
+    <!-- inertial tag goes here (required for gazebo) -->
+    <xacro:box_inertia m="5.0" l="${base_length}" w="${base_width}" h="${base_height}" xyz="0.0 0.0 ${base_height/2.0}" rpy="0.0 0.0 0.0" />
   </link>
   <!-- When you have at least 2 links, TF is generated -->
@@ -42,4 +44,5 @@
         <material name="grey" />
       </visual>
+      <xacro:cylinder_inertia m="1.0" radius="${wheel_radius}" length="${wheel_length}" xyz="0 0 0" rpy="${ pi / 2.0 } 0 0" />
     </link>
   </xacro:macro>
@@ -54,4 +57,5 @@
       <material name="grey" />
     </visual>
+    <xacro:sphere_inertia m="0.5" radius="${wheel_radius/2.0}" xyz="0 0 0" rpy="0 0 0" />
   </link>
   <!-- We have to provide joints -->
