Commit message: add macro

File: my_robot_description/urdf/mobile_base.xacro (robot description, xacro)
@@ -33,22 +33,17 @@
     </visual>
   </link>
-  <link name="right_wheel_link">
-    <visual>
-      <geometry>
-        <cylinder radius="${wheel_radius}" length="${wheel_length}" />
-      </geometry>
-      <origin xyz="0 0 0" rpy="${ pi / 2.0 } 0 0" />
-      <material name="grey" />
-    </visual>
-  </link>
-  <link name="left_wheel_link">
-    <visual>
-      <geometry>
-        <cylinder radius="${wheel_radius}" length="${wheel_length}" />
-      </geometry>
-      <origin xyz="0 0 0" rpy="${ pi / 2.0 } 0 0" />
-      <material name="grey" />
-    </visual>
-  </link>
+  <xacro:macro name="wheel_link" params="prefix">
+    <link name="${prefix}_wheel_link">
+      <visual>
+        <geometry>
+          <cylinder radius="${wheel_radius}" length="${wheel_length}" />
+        </geometry>
+        <origin xyz="0 0 0" rpy="${ pi / 2.0 } 0 0" />
+        <material name="grey" />
+      </visual>
+    </link>
+  </xacro:macro>
+  <xacro:wheel_link prefix="left" />
+  <xacro:wheel_link prefix="right" />
   <link name="caster_wheel_link">
     <visual>

Commit message: add collision tags to urdf for gazebo

File: my_robot_description/urdf/mobile_base.xacro (robot description, xacro)
@@ -22,4 +22,10 @@
       <material name="blue" />
     </visual>
+    <collision>
+      <geometry>
+        <box size="${base_length} ${base_width} ${base_height}" />
+      </geometry>
+      <origin xyz="0 0 ${base_height/2.0}" rpy="0 0 0" />
+    </collision>
     <!-- inertial tag goes here (required for gazebo) -->
     <xacro:box_inertia m="5.0" l="${base_length}" w="${base_width}" h="${base_height}" xyz="0.0 0.0 ${base_height/2.0}" rpy="0.0 0.0 0.0" />
@@ -34,4 +40,10 @@
       <material name="grey" />
     </visual>
+    <collision>
+      <geometry>
+        <cylinder radius="0.1" length="0.2" />
+      </geometry>
+      <origin xyz="0 0 0.1" rpy="0 0 0" />
+    </collision>
   </link>
   <xacro:macro name="wheel_link" params="prefix">
@@ -44,4 +56,10 @@
         <material name="grey" />
       </visual>
+      <collision>
+        <geometry>
+          <cylinder radius="${wheel_radius}" length="${wheel_length}" />
+        </geometry>
+        <origin xyz="0 0 0" rpy="${ pi / 2.0 } 0 0" />
+      </collision>
       <xacro:cylinder_inertia m="1.0" radius="${wheel_radius}" length="${wheel_length}" xyz="0 0 0" rpy="${ pi / 2.0 } 0 0" />
     </link>
@@ -57,4 +75,10 @@
       <material name="grey" />
     </visual>
+    <collision>
+      <geometry>
+        <sphere radius="${wheel_radius/2.0}" />
+      </geometry>
+      <origin xyz="0 0 0" rpy="0 0 0" />
+    </collision>
     <xacro:sphere_inertia m="0.5" radius="${wheel_radius/2.0}" xyz="0 0 0" rpy="0 0 0" />
   </link>

Commit message: update launch file to launch gazebo with a world

File: my_robot_description/urdf/mobile_base.xacro (robot description, xacro)
@@ -32,20 +32,4 @@
     <xacro:box_inertia m="5.0" l="${4*base_length}" w="${4*base_width}" h="${4*base_height}" xyz="0.0 0.0 ${base_height/2.0}" rpy="0.0 0.0 0.0" />
   </link>
-  <!-- When you have at least 2 links, TF is generated -->
-  <link name="second_link">
-    <visual>
-      <geometry>
-        <cylinder radius="0.1" length="0.2" />
-      </geometry>
-      <origin xyz="0 0 0.1" rpy="0 0 0" />
-      <material name="grey" />
-    </visual>
-    <collision>
-      <geometry>
-        <cylinder radius="0.1" length="0.2" />
-      </geometry>
-      <origin xyz="0 0 0.1" rpy="0 0 0" />
-    </collision>
-  </link>
   <xacro:macro name="wheel_link" params="prefix">
     <link name="${prefix}_wheel_link">
@@ -66,4 +50,5 @@
     </link>
   </xacro:macro>
+  <!-- When you have at least 2 links, TF is generated -->
   <xacro:wheel_link prefix="left" />
   <xacro:wheel_link prefix="right" />
@@ -91,22 +76,16 @@
   </joint>
   <!-- name= {parentLink}_{childLink}_joint (just a convention to keep things consistent, not a necessity) -->
-  <joint name="base_second_joint" type="revolute">
+  <!-- base-right_wheel joint -->
+  <joint name="base_right_wheel_joint" type="continuous">
     <!-- [type="continuous"]= revolute but with no limits -->
     <!-- 4 most common joint types= fixed, revolute, continuous, prismatic -->
     <parent link="base_link" />
-    <child link="second_link" />
+    <child link="right_wheel_link" />
     <!-- ! tip for beginners= put 0 to everything first, then modify by observing the positions at RViz -->
-    <origin xyz="0 0 0.2" rpy="0 0 0" />
+    <origin xyz="${-base_length / 4.0} ${-(base_width / 2.0 + (wheel_length / 2.0))} 0" rpy="0 0 0" />
     <!-- 0= no rotation, 1= +rotation, -1= -rotation -->
-    <axis xyz="0 0 1" />
+    <axis xyz="0 1 0" />
     <!-- lower, upper limits= required for [type="revolute"] (in radians) -->
-    <limit lower="-${ pi / 2.0 }" upper="${ pi / 2.0 }" velocity="100" effort="100" />
-  </joint>
-  <!-- base-right_wheel joint -->
-  <joint name="base_right_wheel_joint" type="continuous">
-    <parent link="base_link" />
-    <child link="right_wheel_link" />
-    <origin xyz="${-base_length / 4.0} ${-(base_width / 2.0 + (wheel_length / 2.0))} 0" rpy="0 0 0" />
-    <axis xyz="0 1 0" />
+    <!-- <limit lower="-${ pi / 2.0 }" upper="${ pi / 2.0 }" velocity="100" effort="100" /> -->
   </joint>
   <!-- base-left_wheel joint -->

File: my_robot_description/urdf/mobile_base_gazebo.xacro (robot description, xacro)
@@ -12,7 +12,33 @@
   <gazebo reference="caster_wheel_link">
     <material>Gazebo/Grey</material>
+    <!-- these lines are about friction (coefficients) -->
+    <mu1 value="0.1" />
+    <mu2 value="0.1" />
   </gazebo>
-  <gazebo reference="second_link">
-    <material>Gazebo/Green</material>
+  <!-- diff drive plugin -->
+  <gazebo>
+    <plugin name="diff_drive_controller" filename="libgazebo_ros_diff_drive.so">
+      <!-- Update rate in Hz -->
+      <update_rate>50</update_rate>
+      <!-- wheels -->
+      <left_joint>base_left_wheel_joint</left_joint>
+      <right_joint>base_right_wheel_joint</right_joint>
+      <!-- kinematics -->
+      <wheel_separation>${base_width + wheel_length}</wheel_separation>
+      <wheel_diameter>${wheel_radius * 2}</wheel_diameter>
+      <!-- limits -->
+      <!-- <max_wheel_torque>20</max_wheel_torque>
+      <max_wheel_acceleration>1.0</max_wheel_acceleration> -->
+      <!-- input -->
+      <!-- send commands to this topic, robot node will listen to this topic -->
+      <command_topic>cmd_vel</command_topic>
+      <!-- output -->
+      <publish_odom>true</publish_odom>
+      <publish_odom_tf>true</publish_odom_tf>
+      <publish_wheel_tf>true</publish_wheel_tf>
+      <odometry_topic>odom</odometry_topic>
+      <odometry_frame>odom</odometry_frame>
+      <robot_base_frame>base_footprint</robot_base_frame>
+    </plugin>
   </gazebo>
 </robot>
